File: Connectors.kicad_sch (KiCad schematic)
At the start: 4 parts, among them J1 Conn_01x04_Pin, J2 Conn_01x04_Pin, J3 Conn_01x09_Pin, J4 Conn_02x03_Odd_Even

Commit message: Updated
Connections:
- net SCK: no longer J1.4 (Pin_4)
- new net SCL: J1.4 (Pin_4)
Changed lines of the file:
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@@
 		)
 	)
-	(hierarchical_label "SCK"
+	(hierarchical_label "SCL"
 		(shape passive)
 		(at 90.17 71.12 0)
