File: MCU DATALOGGER.kicad_sch (KiCad schematic)
At the start: 25 parts, among them U1 24LC1025, U2 24LC1025, U4 ATMEGA328P-AU, U5 DS1337S_, Y1 32.768 KHz, Y2 16 MHz

Commit message: Updated
Connections:
- net SCK: no longer R3.2, U1.6 (SCL), U2.6 (SCL), U4.28 (PC5), U5.6 (SCL)
- new net SCL: R3.2, U1.6 (SCL), U2.6 (SCL), U4.28 (PC5), U5.6 (SCL)
Other:
- sheet Connectors ports: added SCL; removed none
